File: pcb & electronic files/kicad files/keyboard.kicad_pcb (KiCad board)
At the start: 2 copper layers, 295.8 x 148.5 mm, 188 parts, among them J1 AVR-ISP-6, J2 USB_C_Receptacle_USB2.0, SW1 SW_Push, SW2 SW_Push, U1 ATmega32A-PU

Commit message: changed the pcb
changes some of the files
Other:
- board text added: "J73K PCB V1.1"
- board text removed: "J73K PCB"
